Commit message: Fixed link/joint names and added simulation capabilities

File: manos_description/urdf/grippers/schunk_pg70.gazebo.xacro (robot description, xacro)
@@ -6,9 +6,9 @@
       <self_collide>false</self_collide>
     </gazebo>
-    <gazebo reference="${name}_finger_left_link">
+    <gazebo reference="${name}_finger1_link">
       <gravity>true</gravity>
       <self_collide>false</self_collide>
     </gazebo>
-    <gazebo reference="${name}_finger_right_link">
+    <gazebo reference="${name}_finger2_link">
       <gravity>true</gravity>
       <self_collide>false</self_collide>

File: manos_description/urdf/grippers/schunk_pg70.transmission.xacro (robot description, xacro)
@@ -3,20 +3,20 @@
   <xacro:macro name="schunk_pg70_transmission" params="name">
     <!-- finger1 -->
-    <transmission name="${name}_finger_left_trans">
+    <transmission name="${name}_finger1_trans">
       <type>transmission_interface/SimpleTransmission</type>
-      <joint name="${name}_finger_left_joint">
-        <hardwareInterface>PositionJointInterface</hardwareInterface>
+      <joint name="${name}_finger1_joint">
+        <hardwareInterface>hardware_interface/PositionJointInterface</hardwareInterface>
       </joint>
-      <actuator name="${name}_finger_left_motor">
+      <actuator name="${name}_finger1_motor">
         <mechanicalReduction>1</mechanicalReduction>
       </actuator>
     </transmission>
     <!-- finger2 -->
-    <transmission name="${name}_finger_right_trans">
+    <transmission name="${name}_finger2_trans">
       <type>transmission_interface/SimpleTransmission</type>
-      <joint name="${name}_finger_right_joint">
-        <hardwareInterface>PositionJointInterface</hardwareInterface>
+      <joint name="${name}_finger2_joint">
+        <hardwareInterface>hardware_interface/PositionJointInterface</hardwareInterface>
       </joint>
-      <actuator name="${name}_finger_right_motor">
+      <actuator name="${name}_finger2_motor">
         <mechanicalReduction>1</mechanicalReduction>
       </actuator>

File: manos_description/urdf/grippers/schunk_pg70.urdf.xacro (robot description, xacro)
@@ -24,5 +24,5 @@
           <mesh filename="package://schunk_pg70/meshes/pg70.dae" />
         </geometry>
-    <material name="blue"/>
+        <material name="blue"/>
       </collision>
       <inertia>
@@ -33,12 +33,12 @@
     </link>
 <!-- LEFT FINGER BASE -->
-    <joint name="${name}_finger_left_joint" type="prismatic" >
+    <joint name="${name}_finger1_joint" type="prismatic" >
       <parent link="${name}_base_link" />
-      <child link="${name}_finger_left_link" />
+      <child link="${name}_finger1_link" />
       <limit effort="100" lower="-0.001" upper="0.04" velocity="2.0"/>
-      <origin xyz="0 0 0.0789" rpy="0 0 0"/>
+      <origin xyz="0 0.03 0.0789" rpy="0 0 0"/>
       <axis xyz="0 1 0" />
     </joint>
-    <link name="${name}_finger_left_link">
+    <link name="${name}_finger1_link">
       <visual>
         <geometry>
@@ -53,5 +53,5 @@
           <box size="0.03 0.01 0.01"/>
         </geometry>
-    <material name="black" />
+        <material name="black" />
       </collision>
        <inertial> <origin xyz="0 0 0" rpy="0 0 0"/> <mass value="1"/> <inertia ixx="1.0" ixy="0.0" ixz="0.0" iyy="1.0" iyz="0.0" izz="1.0"/> </inertial>
@@ -59,5 +59,5 @@
 <!-- LEFT FINGERTIP -->
     <joint name="${name}_fingertip_left_joint" type="fixed" >
-      <parent link="${name}_finger_left_link" />
+      <parent link="${name}_finger1_link" />
       <child link="${name}_fingertip_left_link" />
       <origin xyz="0.015 -0.001 0.045" rpy="${pi/2} 0 -${pi/2}"/>
@@ -76,17 +76,17 @@
           <mesh filename="package://manos_description/meshes/schunk_pg70/finger.stl" />
         </geometry>
-           <material name="black"/>
+        <material name="black"/>
       </collision>
     </link>
 <!-- RIGHT FINGER BASE -->
-    <joint name="${name}_finger_right_joint" type="prismatic" >
-      <mimic joint="${name}_finger_left_joint" multiplier="1" offset="0"/>
+    <joint name="${name}_finger2_joint" type="prismatic" >
+      <mimic joint="${name}_finger1_joint" multiplier="1" offset="0"/>
       <parent link="${name}_base_link" />
-      <child link="${name}_finger_right_link" />
+      <child link="${name}_finger2_link" />
       <limit effort="100" lower="-0.001" upper="0.04" velocity="2.0"/>
-      <origin xyz="0 0 0.0789" rpy="-0 0 0"/>
+      <origin xyz="0 -0.03 0.0789" rpy="-0 0 0"/>
       <axis xyz="0 -1 0" />
     </joint>
-    <link name="${name}_finger_right_link">
+    <link name="${name}_finger2_link">
       <visual>
         <geometry>
@@ -99,5 +99,5 @@
           <box size="0.03 0.01 0.01"/>
         </geometry>
-    <material name="black"/>
+        <material name="black"/>
       </collision>
        <inertial> <origin xyz="0 0 0" rpy="0 0 0"/> <mass value="1"/> <inertia ixx="1.0" ixy="0.0" ixz="0.0" iyy="1.0" iyz="0.0" izz="1.0"/> </inertial>
@@ -105,5 +105,5 @@
 <!-- RIGHT FINGERTIP -->
     <joint name="${name}_fingertip_right_joint" type="fixed" >
-      <parent link="${name}_finger_right_link" />
+      <parent link="${name}_finger2_link" />
       <child link="${name}_fingertip_right_link" />
      <origin xyz="-0.015 0.001 0.045" rpy="${pi/2} 0 ${pi/2}"/>
@@ -120,5 +120,5 @@
           <mesh filename="package://manos_description/meshes/schunk_pg70/finger.stl" />
         </geometry>
-    <material name="black"/>
+        <material name="black"/>
      </collision>
     </link>

File: manos_description/urdf/ur3_pg70.urdf.xacro (robot description, xacro)
@@ -61,5 +61,5 @@
  </joint>
   <!-- GRIPPER -->
-  <xacro:schunk_pg70 name="schunk_pg70" parent="gripper_link">
+  <xacro:schunk_pg70 name="pg70" parent="gripper_link">
     <origin xyz="0 0.0 0.0091" rpy="0 0 0" /> <!--slightly above gazebo plane-->
   </xacro:schunk_pg70>
@@ -107,5 +107,5 @@
   </link>
   <joint name="gripper_power_joint" type="fixed">
-    <parent link="schunk_pg70_base_link"/>
+    <parent link="pg70_base_link"/>
     <child link="gripper_power_box"/>
     <origin xyz="0.004 -0.08 0.03" rpy="0.0 0.0 ${pi/2}" />

Commit message: Enabled the pg70 simulation!

File: manos_description/urdf/grippers/schunk_pg70.gazebo.xacro (robot description, xacro)
@@ -3,21 +3,16 @@
   <xacro:macro name="schunk_pg70_gazebo" params="name">
     <gazebo reference="${name}_base_link">
-      <gravity>true</gravity>
       <self_collide>false</self_collide>
     </gazebo>
     <gazebo reference="${name}_finger1_link">
-      <gravity>true</gravity>
       <self_collide>false</self_collide>
     </gazebo>
     <gazebo reference="${name}_finger2_link">
-      <gravity>true</gravity>
       <self_collide>false</self_collide>
     </gazebo>
     <gazebo reference="${name}_fingertip_right_link">
-      <gravity>true</gravity>
       <self_collide>false</self_collide>
     </gazebo>
     <gazebo reference="${name}_fingertip_left_link">
-      <gravity>true</gravity>
       <self_collide>false</self_collide>
     </gazebo>

File: manos_description/urdf/grippers/schunk_pg70.urdf.xacro (robot description, xacro)
@@ -10,16 +10,18 @@
       <xacro:insert_block name="origin" />
     </joint>
-  <material name="silver">
-    <color rgba="0.5 0.5 0.5 1"/>
-  </material>
-  <material name="light_silver">
-    <color rgba="0.7 0.7 0.7 1"/>
-  </material>
-  <material name="white">
-    <color rgba="1 1 1 1"/>
-  </material>
-  <material name="black">
-    <color rgba="0 0 0 1"/>
-  </material>
+    <xacro:schunk_pg70_transmission name="${name}"/>
+    <xacro:schunk_pg70_gazebo name="${name}" />
+    <material name="silver">
+      <color rgba="0.5 0.5 0.5 1"/>
+    </material>
+    <material name="light_silver">
+      <color rgba="0.7 0.7 0.7 1"/>
+    </material>
+    <material name="white">
+      <color rgba="1 1 1 1"/>
+    </material>
+    <material name="black">
+      <color rgba="0 0 0 1"/>
+    </material>
 <!--     PALM -->
     <link name="${name}_base_link">
@@ -44,6 +46,6 @@
       <parent link="${name}_base_link" />
       <child link="${name}_finger1_link" />
-      <limit effort="100" lower="-0.001" upper="0.04" velocity="2.0"/>
-      <origin xyz="0 0.04 0.095" rpy="0 0 0"/>
+      <limit effort="100" lower="0.0015" upper="0.04" velocity="2.0"/>
+      <origin xyz="0 0.0015 0.095" rpy="0 0 0"/>
       <axis xyz="0 1 0" />
     </joint>
@@ -87,9 +89,9 @@
 <!-- RIGHT FINGER BASE -->
     <joint name="${name}_finger2_joint" type="prismatic" >
-      <mimic joint="${name}_finger1_joint" multiplier="1" offset="0"/>
+      <!-- <mimic joint="${name}_finger1_joint" multiplier="1" offset="0"/> -->
       <parent link="${name}_base_link" />
       <child link="${name}_finger2_link" />
-      <limit effort="100" lower="-0.001" upper="0.04" velocity="2.0"/>
-      <origin xyz="0 -0.04 0.095" rpy="-0 0 0"/>
+      <limit effort="100" lower="0.0015" upper="0.04" velocity="2.0"/>
+      <origin xyz="0 -0.0015 0.095" rpy="-0 0 0"/>
       <axis xyz="0 -1 0" />
     </joint>
@@ -167,6 +169,4 @@
     <origin xyz="-0.01 -0.042 -0.011" rpy="${pi/2} 0.0 0.0" />
  </joint>
-    <xacro:schunk_pg70_transmission name="${name}"/>
-    <xacro:schunk_pg70_gazebo name="${name}" />
   </xacro:macro>
 </robot>
