Commit message: Updated urdf and .dae files to reflect reality with more accuracy

File: manos_description/urdf/grippers/schunk_pg70.urdf.xacro (robot description, xacro)
@@ -10,25 +10,33 @@
       <xacro:insert_block name="origin" />
     </joint>
+  <material name="silver">
+    <color rgba="0.5 0.5 0.5 1"/>
+  </material>
+  <material name="light_silver">
+    <color rgba="0.7 0.7 0.7 1"/>
+  </material>
+  <material name="white">
+    <color rgba="1 1 1 1"/>
+  </material>
+  <material name="black">
+    <color rgba="0 0 0 1"/>
+  </material>
 <!--     PALM -->
     <link name="${name}_base_link">
       <visual>
         <geometry>
-          <mesh filename="package://schunk_pg70/meshes/pg70.dae" />
+          <mesh filename="package://manos_description/meshes/schunk_pg70/pg70.dae" />
         </geometry>
-        <material name="blue">
-          <color rgba="0 0 1 1"/>
-        </material>
       </visual>
       <collision>
         <geometry>
-          <mesh filename="package://schunk_pg70/meshes/pg70.dae" />
+          <mesh filename="package://manos_description/meshes/schunk_pg70/pg70.dae" />
         </geometry>
-        <material name="blue"/>
       </collision>
-      <inertia>
+      <inertial>
           <origin xyz="0.000019 -0.000347 0.028892"/>
-         <mass value="0.0"/>
+         <mass value="2.0"/>
          <inertia ixx="0.000002" ixy="0.0" ixz="0.0" iyy="0.000001" iyz="0.0" izz="0.000002"/>
-      </inertia>
+      </inertial>
     </link>
 <!-- LEFT FINGER BASE -->
@@ -45,7 +53,5 @@
           <box size="0.03 0.01 0.01"/>
         </geometry>
-        <material name="black">
-          <color rgba="0 0 0 1"/>
-        </material>
+        <material name="black"/>
       </visual>
       <collision>
@@ -53,7 +59,6 @@
           <box size="0.03 0.01 0.01"/>
         </geometry>
-        <material name="black" />
       </collision>
-       <inertial> <origin xyz="0 0 0" rpy="0 0 0"/> <mass value="1"/> <inertia ixx="1.0" ixy="0.0" ixz="0.0" iyy="1.0" iyz="0.0" izz="1.0"/> </inertial>
+       <!-- <inertial> <origin xyz="0 0 0" rpy="0 0 0"/> <mass value="1"/> <inertia ixx="1.0" ixy="0.0" ixz="0.0" iyy="1.0" iyz="0.0" izz="1.0"/> </inertial> -->
     </link>
 <!-- LEFT FINGERTIP -->
@@ -68,7 +73,5 @@
           <mesh filename="package://manos_description/meshes/schunk_pg70/finger.stl" />
         </geometry>
-        <material name="silver">
-          <color rgba="0.8 0.8 0.8 1"/>
-        </material>
+        <material name="white"/>
       </visual>
       <collision>
@@ -76,5 +79,4 @@
           <mesh filename="package://manos_description/meshes/schunk_pg70/finger.stl" />
         </geometry>
-        <material name="black"/>
       </collision>
     </link>
@@ -93,5 +95,5 @@
           <box size="0.03 0.01 0.01"/>
         </geometry>
-    <material name="black"/>
+      <material name="black"/>
       </visual>
       <collision>
@@ -99,7 +101,6 @@
           <box size="0.03 0.01 0.01"/>
         </geometry>
-        <material name="black"/>
       </collision>
-       <inertial> <origin xyz="0 0 0" rpy="0 0 0"/> <mass value="1"/> <inertia ixx="1.0" ixy="0.0" ixz="0.0" iyy="1.0" iyz="0.0" izz="1.0"/> </inertial>
+       <!-- <inertial> <origin xyz="0 0 0" rpy="0 0 0"/> <mass value="1"/> <inertia ixx="1.0" ixy="0.0" ixz="0.0" iyy="1.0" iyz="0.0" izz="1.0"/> </inertial> -->
     </link>
 <!-- RIGHT FINGERTIP -->
@@ -114,5 +115,5 @@
           <mesh filename="package://manos_description/meshes/schunk_pg70/finger.stl" />
         </geometry>
-    <material name="silver" />
+      <material name="white" />
       </visual>
       <collision>
@@ -120,7 +121,42 @@
           <mesh filename="package://manos_description/meshes/schunk_pg70/finger.stl" />
         </geometry>
-        <material name="black"/>
      </collision>
     </link>
+         <link name="gripper_power_cable">
+    <visual>
+      <geometry>
+        <cylinder length="0.035" radius="0.012"/>
+      </geometry>
+      <material name="light_silver"/>
+    </visual>
+    <collision>
+      <geometry>
+        <cylinder length="0.035" radius="0.012"/>
+      </geometry>
+    </collision>
+ </link>
+  <link name="gripper_power_box">
+    <visual>
+      <geometry>
+        <box size="0.047 0.072 0.072"/>
+      </geometry>
+      <material name="silver"/>
+    </visual>
+    <collision>
+      <geometry>
+       <box size="0.047 0.072 0.072"/>
+      </geometry>
+    </collision>
+  </link>
+  <joint name="gripper_power_joint" type="fixed">
+    <parent link="${name}_base_link"/>
+    <child link="gripper_power_box"/>
+    <origin xyz="0.004 -0.08 0.03" rpy="0.0 0.0 ${pi/2}" />
+ </joint>
+ <joint name="gripper_power_cable_joint" type="fixed">
+    <parent link="gripper_power_box"/>
+    <child link="gripper_power_cable"/>
+    <origin xyz="-0.01 -0.042 -0.011" rpy="${pi/2} 0.0 0.0" />
+ </joint>
     <xacro:schunk_pg70_transmission name="${name}"/>
     <xacro:schunk_pg70_gazebo name="${name}" />

File: manos_description/urdf/ur3_pg70.urdf.xacro (robot description, xacro)
@@ -40,6 +40,6 @@
         <box size="0.08 0.113 0.005"/>
       </geometry>
-      <material name="o">
-        <color rgba="0.549019608 0.450980392 0.235294118 1" />
+      <material name="silver">
+        <color rgba="0.5 0.5 0.5 1" />
       </material>
     </visual>
@@ -64,51 +64,4 @@
     <origin xyz="0 0.0 0.0091" rpy="0 0 0" /> <!--slightly above gazebo plane-->
   </xacro:schunk_pg70>
- <link name="gripper_power_cable">
-    <visual>
-      <geometry>
-        <cylinder length="0.035" radius="0.012"/>
-      </geometry>
-      <material name="o">
-         <color rgba="0.549019608 0.450980392 0.235294118 1" />
-      </material>
-    </visual>
-    <inertial>
-        <origin xyz="0 0 0" rpy="0 0 0"/>
-        <mass value="0.01"/>
-        <inertia ixx="0.0001" ixy="0" ixz="0" iyy="0.0001" iyz="0" izz="0.0001" />
-    </inertial>
-    <collision>
-      <geometry>
-        <cylinder length="0.035" radius="0.012"/>
-      </geometry>
-    </collision>
- </link>
- <joint name="gripper_power_cable_joint" type="fixed">
-    <parent link="gripper_power_box"/>
-    <child link="gripper_power_cable"/>
-    <origin xyz="-0.01 -0.042 -0.011" rpy="${pi/2} 0.0 0.0" />
- </joint>
-  <link name="gripper_power_box">
-    <visual>
-      <geometry>
-        <box size="0.047 0.072 0.072"/>
-         <material
-        name="">
-        <color
-          rgba="0.549019608 0.450980392 0.235294118 1" />
-      </material>
-      </geometry>
-    </visual>
-    <collision>
-      <geometry>
-       <box size="0.047 0.072 0.072"/>
-      </geometry>
-    </collision>
-  </link>
-  <joint name="gripper_power_joint" type="fixed">
-    <parent link="pg70_base_link"/>
-    <child link="gripper_power_box"/>
-    <origin xyz="0.004 -0.08 0.03" rpy="0.0 0.0 ${pi/2}" />
- </joint>
  <!--<joint name="ar_marker_joint" type="fixed">
     <parent link="base_link"/>

Commit message: Improved the overall accuracy of the urdf

File: manos_description/urdf/grippers/schunk_pg70.urdf.xacro (robot description, xacro)
@@ -45,5 +45,5 @@
       <child link="${name}_finger1_link" />
       <limit effort="100" lower="-0.001" upper="0.04" velocity="2.0"/>
-      <origin xyz="0 0.03 0.0789" rpy="0 0 0"/>
+      <origin xyz="0 0.04 0.095" rpy="0 0 0"/>
       <axis xyz="0 1 0" />
     </joint>
@@ -87,5 +87,5 @@
       <child link="${name}_finger2_link" />
       <limit effort="100" lower="-0.001" upper="0.04" velocity="2.0"/>
-      <origin xyz="0 -0.03 0.0789" rpy="-0 0 0"/>
+      <origin xyz="0 -0.04 0.095" rpy="-0 0 0"/>
       <axis xyz="0 -1 0" />
     </joint>
@@ -152,5 +152,5 @@
     <parent link="${name}_base_link"/>
     <child link="gripper_power_box"/>
-    <origin xyz="0.004 -0.08 0.03" rpy="0.0 0.0 ${pi/2}" />
+    <origin xyz="0.0 -0.08 0.03" rpy="0.0 0.0 ${pi/2}" />
  </joint>
  <joint name="gripper_power_cable_joint" type="fixed">

File: manos_description/urdf/ur3_pg70.urdf.xacro (robot description, xacro)
@@ -38,5 +38,5 @@
     <visual>
       <geometry>
-        <box size="0.08 0.113 0.005"/>
+        <box size="0.005 0.113 0.08 "/>
       </geometry>
       <material name="silver">
@@ -51,5 +51,5 @@
     <collision>
       <geometry>
-        <box size="0.08 0.113 0.005"/>
+        <box size="0.005 0.113 0.08 "/>
       </geometry>
     </collision>
@@ -62,5 +62,5 @@
   <!-- GRIPPER -->
   <xacro:schunk_pg70 name="pg70" parent="gripper_link">
-    <origin xyz="0 0.0 0.0091" rpy="${pi} -${pi/2} 0" /> <!--slightly above gazebo plane-->
+    <origin xyz="0.0095 0 0" rpy="${pi} -${pi/2} 0" />
   </xacro:schunk_pg70>
  <!--<joint name="ar_marker_joint" type="fixed">

Commit message: Added inertial tag for simulation purposes

File: manos_description/urdf/grippers/schunk_pg70.urdf.xacro (robot description, xacro)
@@ -60,5 +60,9 @@
         </geometry>
       </collision>
-       <!-- <inertial> <origin xyz="0 0 0" rpy="0 0 0"/> <mass value="1"/> <inertia ixx="1.0" ixy="0.0" ixz="0.0" iyy="1.0" iyz="0.0" izz="1.0"/> </inertial> -->
+      <inertial>
+          <origin xyz="0.0 0.0 0.0"/>
+         <mass value="0.2"/>
+         <inertia ixx="1.0" ixy="0.0" ixz="0.0" iyy="1.0" iyz="0.0" izz="1.0"/>
+      </inertial>
     </link>
 <!-- LEFT FINGERTIP -->
@@ -102,5 +106,9 @@
         </geometry>
       </collision>
-       <!-- <inertial> <origin xyz="0 0 0" rpy="0 0 0"/> <mass value="1"/> <inertia ixx="1.0" ixy="0.0" ixz="0.0" iyy="1.0" iyz="0.0" izz="1.0"/> </inertial> -->
+      <inertial>
+          <origin xyz="0.0 0.0 0.0"/>
+         <mass value="0.2"/>
+         <inertia ixx="1.0" ixy="0.0" ixz="0.0" iyy="1.0" iyz="0.0" izz="1.0"/>
+      </inertial>
     </link>
 <!-- RIGHT FINGERTIP -->

Commit message: Added a center gripper link, for better graspit compatibility

File: manos_description/urdf/grippers/schunk_pg70.urdf.xacro (robot description, xacro)
@@ -42,4 +42,10 @@
       </inertial>
     </link>
+  <link name="${name}_center_link"/>
+  <joint name="${name}_center_joint" type="fixed">
+    <parent link="${name}_base_link"/>
+    <child link="${name}_center_link"/>
+    <origin xyz="0 0 0.04903" rpy="0.0 0.0 0.0" />
+ </joint>
 <!-- LEFT FINGER BASE -->
     <joint name="${name}_finger1_joint" type="prismatic" >
