Commit message: Removed unnecessary declarations from limited version too

File: manos_description/urdf/ur3_pg70_limited.urdf.xacro (robot description, xacro)
@@ -71,16 +71,3 @@
     <origin xyz="0.0095 0 0" rpy="${pi} -${pi/2} 0" />
   </xacro:schunk_pg70>
- <!--<joint name="ar_marker_joint" type="fixed">
-    <parent link="base_link"/>
-    <child link="ar_marker_link"/>
-    <origin xyz="-0.41 0.41 0.00" rpy="0.0 0.0 0.0" />
- </joint>
- <link name="ar_marker_link">
-  </link>-->
-  <gazebo>
-      <plugin name="gazebo_ros_control" filename="libgazebo_ros_control.so">
-        <!--<robotNamespace>ur3_pg70</robotNamespace>-->
-         <robotSimType>gazebo_ros_control/DefaultRobotHWSim</robotSimType>
-      </plugin>
-  </gazebo>
 </robot>

Commit message: Bunch of changes

File: manos_description/urdf/ur3_pg70_limited.urdf.xacro (robot description, xacro)
@@ -42,4 +42,22 @@
     <origin xyz="0.0 0.0 0.43" rpy="0 0 1.57" />
  </joint>
+<link name="FT300_link">
+    <visual>
+      <geometry>
+        <cylinder length="0.04" radius="0.035"/>
+      </geometry>
+      <material name="black"/>
+    </visual>
+    <collision>
+      <geometry>
+        <cylinder length="0.04" radius="0.035"/>
+      </geometry>
+    </collision>
+   </link>
+  <joint name="FT300_joint" type="fixed">
+    <origin xyz="0.02 0 0" rpy="0 1.57 0" />
+    <parent link="ee_link" />
+    <child link="FT300_link" />
+  </joint>
  <!--  <link name="gripper_link">
     <visual>

Commit message: Updates in the reactive framework

File: manos_description/urdf/ur3_pg70_limited.urdf.xacro (robot description, xacro)
@@ -43,5 +43,5 @@
     <origin xyz="0.0 0.0 0.43" rpy="0 0 1.57" />
  </joint>
-<link name="FT300_link">
+<!-- <link name="FT300_link">
     <visual>
       <geometry>
@@ -61,4 +61,5 @@
     <child link="FT300_link" />
   </joint>
+ -->
  <!--  <link name="gripper_link">
     <visual>

Commit message: minor commits

File: manos_description/urdf/ur3_pg70_limited.urdf.xacro (robot description, xacro)
@@ -43,5 +43,5 @@
     <origin xyz="0.0 0.0 0.43" rpy="0 0 1.57" />
  </joint>
-<link name="FT300_link">
+<!-- <link name="FT300_link">
     <visual>
       <geometry>
@@ -60,5 +60,5 @@
     <parent link="ee_link" />
     <child link="FT300_link" />
-  </joint>
+  </joint> -->
  <!--  <link name="gripper_link">
     <visual>
