Commit message: Added bringup package and fixed description. Some files might not be needed. I will clean up. Alright?

File: manos_description/urdf/ur3_pg70.urdf.xacro (robot description, xacro)
@@ -3,5 +3,5 @@
   name="ur3_pg70">
 <!-- schunk_pg70 -->
-  <xacro:include filename="$(find schunk_pg70)/urdf/pg70.urdf.xacro"/>
+  <xacro:include filename="$(find manos_description)/urdf/grippers/schunk_pg70.urdf.xacro"/>
 <!-- ur3 -->
   <xacro:include filename="$(find ur_description)/urdf/ur3.urdf.xacro" />
@@ -111,5 +111,5 @@
     <origin xyz="0.004 -0.08 0.03" rpy="0.0 0.0 ${pi/2}" />
  </joint>
- <joint name="ar_marker_joint" type="fixed">
+ <!--<joint name="ar_marker_joint" type="fixed">
     <parent link="base_link"/>
     <child link="ar_marker_link"/>
@@ -117,5 +117,5 @@
  </joint>
  <link name="ar_marker_link">
-  </link>
+  </link>-->
   <gazebo>
       <plugin name="gazebo_ros_control" filename="libgazebo_ros_control.so">

Commit message: Matched gripper_link with ee_link rotation

File: manos_description/urdf/ur3_pg70.urdf.xacro (robot description, xacro)
@@ -58,5 +58,5 @@
     <parent link="ee_link"/>
     <child link="gripper_link"/>
-    <origin xyz="0.0 0.0 0.0" rpy="${pi} -${pi/2} 0.0" />
+    <origin xyz="0.0 0.0 0.0" rpy="0.0 0.0 0.0" />
  </joint>
   <!-- GRIPPER -->

Commit message: Matched gripper_link with ee_link rotation and it's working

File: manos_description/urdf/ur3_pg70.urdf.xacro (robot description, xacro)
@@ -62,5 +62,5 @@
   <!-- GRIPPER -->
   <xacro:schunk_pg70 name="pg70" parent="gripper_link">
-    <origin xyz="0 0.0 0.0091" rpy="0 0 0" /> <!--slightly above gazebo plane-->
+    <origin xyz="0 0.0 0.0091" rpy="${pi} -${pi/2} 0" /> <!--slightly above gazebo plane-->
   </xacro:schunk_pg70>
  <!--<joint name="ar_marker_joint" type="fixed">

Commit message: Removed unnecessary declarations

File: manos_description/urdf/ur3_pg70.urdf.xacro (robot description, xacro)
@@ -64,16 +64,3 @@
     <origin xyz="0.0095 0 0" rpy="${pi} -${pi/2} 0" />
   </xacro:schunk_pg70>
- <!--<joint name="ar_marker_joint" type="fixed">
-    <parent link="base_link"/>
-    <child link="ar_marker_link"/>
-    <origin xyz="-0.41 0.41 0.00" rpy="0.0 0.0 0.0" />
- </joint>
- <link name="ar_marker_link">
-  </link>-->
-  <gazebo>
-      <plugin name="gazebo_ros_control" filename="libgazebo_ros_control.so">
-        <!--<robotNamespace>ur3_pg70</robotNamespace>-->
-         <robotSimType>gazebo_ros_control/DefaultRobotHWSim</robotSimType>
-      </plugin>
-  </gazebo>
 </robot>

Commit message: controllers update

File: manos_description/urdf/ur3_pg70.urdf.xacro (robot description, xacro)
@@ -35,5 +35,5 @@
     <origin xyz="0.0 0.0 0.43" rpy="0 0 1.57" />
  </joint>
-  <link name="gripper_link">
+<!--   <link name="gripper_link">
     <visual>
       <geometry>
@@ -60,8 +60,10 @@
     <origin xyz="0.0 0.0 0.0" rpy="0.0 0.0 0.0" />
  </joint>
+ -->
   <!-- GRIPPER -->
-  <xacro:schunk_pg70 name="pg70" parent="gripper_link">
+<!--   <xacro:schunk_pg70 name="pg70" parent="gripper_link">
     <origin xyz="0.0095 0 0" rpy="${pi} -${pi/2} 0" />
   </xacro:schunk_pg70>
+ -->
   <gazebo>
       <plugin name="gazebo_ros_control" filename="libgazebo_ros_control.so">

File: manos_description/urdf/ur3_pg70_limited.urdf.xacro (robot description, xacro)
@@ -3,5 +3,5 @@
   name="ur3_pg70">
 <!-- schunk_pg70 -->
-  <xacro:include filename="$(find manos_description)/urdf/grippers/schunk_pg70.urdf.xacro"/>
+  <!-- <xacro:include filename="$(find manos_description)/urdf/grippers/schunk_pg70.urdf.xacro"/> -->
 <!-- ur3 -->
   <xacro:include filename="$(find ur_description)/urdf/ur3.urdf.xacro" />
@@ -42,5 +42,5 @@
     <origin xyz="0.0 0.0 0.43" rpy="0 0 1.57" />
  </joint>
-  <link name="gripper_link">
+ <!--  <link name="gripper_link">
     <visual>
       <geometry>
@@ -66,9 +66,10 @@
     <child link="gripper_link"/>
     <origin xyz="0.0 0.0 0.0" rpy="0.0 0.0 0.0" />
- </joint>
+ </joint> -->
   <!-- GRIPPER -->
-  <xacro:schunk_pg70 name="pg70" parent="gripper_link">
+<!--   <xacro:schunk_pg70 name="pg70" parent="gripper_link">
     <origin xyz="0.0095 0 0" rpy="${pi} -${pi/2} 0" />
   </xacro:schunk_pg70>
+ -->
   <gazebo>
       <plugin name="gazebo_ros_control" filename="libgazebo_ros_control.so">

Commit message: updated_driver

File: manos_description/urdf/ur3_pg70.urdf.xacro (robot description, xacro)
@@ -5,7 +5,16 @@
   <xacro:include filename="$(find manos_description)/urdf/grippers/schunk_pg70.urdf.xacro"/>
 <!-- ur3 -->
+  <xacro:arg name="transmission_hw_interface" default="hardware_interface/PositionJointInterface"/>
+  <!-- common stuff -->
+  <xacro:include filename="$(find ur_description)/urdf/common.gazebo.xacro" />
+  <!-- ur3 -->
   <xacro:include filename="$(find ur_description)/urdf/ur3.urdf.xacro" />
-  <xacro:ur3_robot prefix="" joint_limited="false"/>
-   <link name="world" />
+  <!-- arm -->
+  <xacro:arg name="kinematics_config" default="$(find ur_description)/config/ur3_default.yaml"/>
+  <xacro:ur3_robot prefix="" joint_limited="false"
+    transmission_hw_interface="$(arg transmission_hw_interface)"
+    kinematics_file="${load_yaml('$(arg kinematics_config)')}"
+  />
+  <link name="world" />
   <link name="box_link">
     <visual>
@@ -35,5 +44,5 @@
     <origin xyz="0.0 0.0 0.43" rpy="0 0 1.57" />
  </joint>
-<!--   <link name="gripper_link">
+  <link name="gripper_link">
     <visual>
       <geometry>
@@ -60,10 +69,8 @@
     <origin xyz="0.0 0.0 0.0" rpy="0.0 0.0 0.0" />
  </joint>
- -->
   <!-- GRIPPER -->
-<!--   <xacro:schunk_pg70 name="pg70" parent="gripper_link">
+  <xacro:schunk_pg70 name="pg70" parent="gripper_link">
     <origin xyz="0.0095 0 0" rpy="${pi} -${pi/2} 0" />
   </xacro:schunk_pg70>
- -->
   <gazebo>
       <plugin name="gazebo_ros_control" filename="libgazebo_ros_control.so">

File: manos_description/urdf/ur3_pg70_limited.urdf.xacro (robot description, xacro)
@@ -3,9 +3,14 @@
   name="ur3_pg70">
 <!-- schunk_pg70 -->
-  <!-- <xacro:include filename="$(find manos_description)/urdf/grippers/schunk_pg70.urdf.xacro"/> -->
+  <xacro:include filename="$(find manos_description)/urdf/grippers/schunk_pg70.urdf.xacro"/>
 <!-- ur3 -->
-<property name="prefix" value="" />
-  <xacro:include filename="$(find ur_description)/urdf/ur3.urdf.xacro" params="$(prefix) hardware_interface/VelocityJointInterface"/>
-    <xacro:ur3_robot prefix="" joint_limited="true"
+  <xacro:arg name="transmission_hw_interface" default="hardware_interface/PositionJointInterface"/>
+  <!-- common stuff -->
+  <xacro:include filename="$(find ur_description)/urdf/common.gazebo.xacro" />
+  <!-- ur3 -->
+  <xacro:include filename="$(find ur_description)/urdf/ur3.urdf.xacro" />
+  <!-- arm -->
+  <xacro:arg name="kinematics_config" default="$(find ur_description)/config/ur3_default.yaml"/>
+  <xacro:ur3_robot prefix="" joint_limited="true"
     shoulder_pan_lower_limit="${-pi}" shoulder_pan_upper_limit="${pi}"
     shoulder_lift_lower_limit="${-pi}" shoulder_lift_upper_limit="${pi}"
@@ -14,4 +19,6 @@
     wrist_2_lower_limit="${-pi}" wrist_2_upper_limit="${pi}"
     wrist_3_lower_limit="${-pi}" wrist_3_upper_limit="${pi}"
+    transmission_hw_interface="$(arg transmission_hw_interface)"
+    kinematics_file="${load_yaml('$(arg kinematics_config)')}"
   />
    <link name="world" />
@@ -61,5 +68,5 @@
     <child link="FT300_link" />
   </joint> -->
- <!--  <link name="gripper_link">
+  <link name="gripper_link">
     <visual>
       <geometry>
@@ -85,10 +92,9 @@
     <child link="gripper_link"/>
     <origin xyz="0.0 0.0 0.0" rpy="0.0 0.0 0.0" />
- </joint> -->
+ </joint>
   <!-- GRIPPER -->
-<!--   <xacro:schunk_pg70 name="pg70" parent="gripper_link">
+  <xacro:schunk_pg70 name="pg70" parent="gripper_link">
     <origin xyz="0.0095 0 0" rpy="${pi} -${pi/2} 0" />
   </xacro:schunk_pg70>
- -->
   <gazebo>
       <plugin name="gazebo_ros_control" filename="libgazebo_ros_control.so">

File: manos_description/urdf/ur3_table_limited_v2020.urdf.xacro (robot description, xacro)
@@ -2,13 +2,22 @@
 <robot xmlns:xacro="http://wiki.ros.org/xacro"
        name="ur3" >
-  <xacro:arg name="transmission_hw_interface" default="hardware_interface/VelocityJointInterface"/>
+  <xacro:arg name="transmission_hw_interface" default="hardware_interface/PositionJointInterface"/>
+  <!-- common stuff -->
+  <xacro:include filename="$(find ur_description)/urdf/common.gazebo.xacro" />
   <!-- ur3 -->
-  <xacro:include filename="$(find manos_description)/urdf/ur3_control.urdf.xacro" params="$(prefix) hardware_interface/VelocityJointInterface"/>
+  <xacro:include filename="$(find ur_description)/urdf/ur3.urdf.xacro" />
   <!-- arm -->
   <xacro:arg name="kinematics_config" default="$(find ur_description)/config/ur3_default.yaml"/>
-  <xacro:ur3_robot prefix="" joint_limited="false"
+  <xacro:ur3_robot prefix="" joint_limited="true"
+    shoulder_pan_lower_limit="${-pi}" shoulder_pan_upper_limit="${pi}"
+    shoulder_lift_lower_limit="${-pi}" shoulder_lift_upper_limit="${pi}"
+    elbow_joint_lower_limit="${-pi}" elbow_joint_upper_limit="${pi}"
+    wrist_1_lower_limit="${-pi}" wrist_1_upper_limit="${pi}"
+    wrist_2_lower_limit="${-pi}" wrist_2_upper_limit="${pi}"
+    wrist_3_lower_limit="${-pi}" wrist_3_upper_limit="${pi}"
     transmission_hw_interface="$(arg transmission_hw_interface)"
+    kinematics_file="${load_yaml('$(arg kinematics_config)')}"
   />
-   <link name="world" />
+  <link name="world" />
   <link name="box_link">
     <visual>
@@ -38,10 +47,3 @@
     <origin xyz="0.0 0.0 0.43" rpy="0 0 1.57" />
  </joint>
-  <gazebo>
-      <plugin name="gazebo_ros_control" filename="libgazebo_ros_control.so">
-        <robotNamespace>/</robotNamespace>
-        <robotSimType>gazebo_ros_control/DefaultRobotHWSim</robotSimType>
-        <legacyModeNS>true</legacyModeNS>
-      </plugin>
-  </gazebo>
 </robot>

File: manos_description/urdf/ur3_table_v2020.urdf.xacro (robot description, xacro)
@@ -2,5 +2,5 @@
 <robot xmlns:xacro="http://wiki.ros.org/xacro"
        name="ur3" >
-  <xacro:arg name="transmission_hw_interface" default="hardware_interface/VelocityJointInterface"/>
+  <xacro:arg name="transmission_hw_interface" default="hardware_interface/PositionJointInterface"/>
   <!-- common stuff -->
   <xacro:include filename="$(find ur_description)/urdf/common.gazebo.xacro" />
@@ -13,5 +13,5 @@
     kinematics_file="${load_yaml('$(arg kinematics_config)')}"
   />
-   <link name="world" />
+  <link name="world" />
   <link name="box_link">
     <visual>
